File: OSO-BOOK-C1/OSO-BOOK-C1.kicad_sch (KiCad schematic)
At the start: 29 parts, among them J1 JST-PH3, J2 JST-PH3, J3 JST-PH4, Q1 Q_PMOS_GSD, Q2 Q_PMOS_GSD, SW1 SW_SPDT, U1 Pico, U2 OSO-BOOK-C2-01, U3 MEM2075, U4 GD25Q16C

Commit message: #1: Annotate original drawings for understanding
Other:
- note added: "OPTIONAL NOTE: RX/TX and spare GPIOS"
- note added: "STEP 1 NOTE: When shorted, depowers 3.3V of PICO output"
- note added: "STEP 2 NOTE: When shorted this grounds the RUN pin on the PICO and resets the board"
- note added: "STEP 3 NOTE: Disconnects VBATT if VBUS is powered"
- note added: "STEP 3 NOTE: EN2 is GPIO0 and controls power switching of components to 3.3V"
- note added: "STEP 4 NOTE: GPIO"
- note added: "STEP 5 GD25Q16C Firmware flash module"
- note added: "STEP 6 SD card module"
- note added: "STEP 7 Raspberry Pi Pico"
- note added: "STEP 8 NOTE: 24 pin serial HAT adaptor board"
- note added: "STEP 9 NOTE: Battery Holder"
- note removed: "Raspberry Pi Pico"
- title: Open Book Abridged Edition -> Open Book Abridged Edition Annotated
